Commit message: Fixed modularity and implemented WOMBAT movement in Gazebo

File: ros_ws/src/simulation/urdf/parameters.xacro (robot description, xacro)
@@ -10,4 +10,8 @@
 <xacro:property name="casterRadius" value="0.0065"/>
 <xacro:property name="casterMass" value="0.012"/>
+<xacro:property name="origin_right_wheel" value="0.05 -0.09 0.0"/>
+<xacro:property name="origin_left_wheel" value="0.05 0.09 0.0"/>
+<xacro:property name="rpy_right_wheel" value="-${PI/2} 0 0"/>
+<xacro:property name="rpy_left_wheel" value="${PI/2} 0 0"/>
 <xacro:property name="wheelHeight" value="0.01"/>
 <xacro:property name="wheelRadius" value="0.05"/>

File: ros_ws/src/simulation/urdf/wombat.xacro (robot description, xacro)
@@ -3,8 +3,11 @@
 <robot name="WOMBAT" xmlns:xacro="http://www.ros.org/wiki/xacro">
 	<!-- files for gazebo costumization -->
-	<xacro:include filename="$(find simulation)/urdf/materials.xacro" />
 	<xacro:include filename="$(find simulation)/urdf/parameters.xacro" />
 	<xacro:include filename="$(find simulation)/urdf/wombat.gazebo" />
 	<xacro:include filename="$(find simulation)/urdf/macros.xacro" />
+    <xacro:include filename="$(find simulation)/urdf/wheel.xacro"/>
+    <xacro:include filename="$(find simulation)/urdf/camera.xacro"/>
+    <xacro:include filename="$(find simulation)/urdf/lidar.xacro"/>
+    <xacro:include filename="$(find simulation)/urdf/chassis.xacro"/>
 	<!-- Dummy link to fiz robot chassis -->
 	<link name="base_link">
@@ -16,229 +19,12 @@
         <origin xyz="0.0 0.0 ${wheelRadius+0.0010032}" />
 	</joint>
-	<link name="chassis">
-		<pose>0 0 0 0 0 0</pose>
-		<visual>
-			<!-- box only
-      <origin xyz="0 0 0" rpy="0 0 0"/>
-          <geometry>
-          	  <box size="${chassisX} ${chassisY} ${chassisZ}"/>
-          </geometry> -->
-			<!-- with mesh  -->
-			<origin xyz="0 0 0" rpy="${PI/2} 0 ${PI/2}" />
-			<geometry>
-				<mesh filename="file://${mesh_chassis}" />
-			</geometry>
-		</visual>
-		<collision name="collision_chassis">
-			<origin rpy="0 0 0" xyz="0 0 0" />
-			<geometry>
-				<box size="${chassisX} ${chassisY} ${chassisZ}" />
-			</geometry>
-		</collision>
-		<inertial>
-			<mass value="${chassisMass}" />
-			<xacro:box_inertia m="${chassisMass}" x="${chassisX}" y="${chassisY}" z="${chassisZ}" />
-		</inertial>
-		<!-- agregar caster wheel en frame -->
-		<collision>
-			<origin xyz="-0.095 0 ${-0.0435}" rpy="0 0 0" />
-			<geometry>
-				<sphere radius="${casterRadius}" />
-			</geometry>
-			<surface>
-				<friction>
-					<ode>
-						<slip1>0.0</slip1>
-						<slip2>0.0</slip2>
-					</ode>
-				</friction>
-			</surface>
-		</collision>
-		<visual>
-			<origin xyz="-0.095 0 -0.0435" rpy="0 0 0" />
-			<geometry>
-				<sphere radius="${casterRadius}" />
-			</geometry>
-		</visual>
-	</link>
-	<!--RIGHT
-	WHEEL -->
-	<link name="right_wheel">
-		<visual>
-			<origin xyz="0 0 0" rpy="-${PI/2} 0 0" />
-			<geometry>
-				<!-- with mesh-->
-				<mesh filename="file://${mesh_wheel}" />
-				<!-- cylinder only
-	    	<cylinder length="${wheelHeight}" radius="${wheelRadius}"/> -->
-			</geometry>
-		</visual>
-		<collision>
-			<origin xyz="0 0 0 " rpy="-${PI/2} 0 0" />
-			<geometry>
-				<cylinder length="${wheelHeight}" radius="${wheelRadius+0.0010032}" />
-			</geometry>
-		</collision>
-		<inertial>
-			<mass value="${wheelMass}" />
-			<origin xyz="0 0 0" rpy="${PI/2} 0 0" />
-			<xacro:wheel_inertia r="${wheelRadius}" l="${wheelHeight}" m="${wheelMass}" />
-		</inertial>
-	</link>
-	<!-- LEFT WHEEL -->
-	<link name="left_wheel">
-		<visual>
-			<geometry>
-				<!-- with mesh-->
-				<mesh filename="file://${mesh_wheel}" />
-				<!-- cylinder only
-	    	<cylinder length="${wheelHeight}" radius="${wheelRadius}"/> -->
-			</geometry>
-			<origin xyz="0 0 0" rpy="${PI/2} 0 0" />
-		</visual>
-		<collision>
-			<origin xyz="0 0 0" rpy="${PI/2} 0 0" />
-			<geometry>
-				<cylinder length="${wheelHeight}" radius="${wheelRadius+0.0010032}" />
-			</geometry>
-		</collision>
-		<inertial>
-			<mass value="${wheelMass}" />
-			<origin xyz="0 0 0" rpy="${PI/2} 0 0" />
-			<xacro:wheel_inertia r="${wheelRadius}" l="${wheelHeight}" m="${wheelMass}" />
-		</inertial>
-	</link>
-	<!-- CAMERA-->
-	<link name="camera">
-		<inertial>
-			<origin rpy="0 0 0" xyz="0 0 0" />
-			<mass value="0.007" />
-			<inertia ixx="0.166667" ixy="0" ixz="0" iyy="0.166667" iyz="0" izz="0.166667" />
-			<!-- ad camera inertia -->
-		</inertial>
-		<collision name="collision_chassis">
-			<origin rpy="0 0 0" xyz="0 0 0" />
-			<geometry>
-				<box size="0.07 0.01 0.06" />
-			</geometry>
-		</collision>
-		<visual>
-			<!-- box only
-		    	    <origin rpy="$0 0 ${PI/2}" xyz="0 0 0"/>
-		          <geometry>
-		          	<box size="0.05 0.01 0.06" />
-		          </geometry>-->
-			<!-- with mesh-->
-			<origin rpy="${PI/2} 0 ${PI/2}" xyz="0 0 0" />
-			<geometry>
-				<mesh filename="file://${mesh_camera}" />
-			</geometry>
-		</visual>
-	</link>
-	<link name="camera_frame_optical" />
-	<!-- LIDAR-->
-	<link name="lidar">
-		<inertial>
-			<mass value="0.1" />
-			<origin xyz="0 0 0" />
-			<inertia ixx="0.01" ixy="0.0" ixz="0.0"
-					 iyy="0.01" iyz="0.0"
-					 izz="0.01" />
-		</inertial>
-		<!-- <visual>
-			<origin xyz=" 0 0 0 " rpy="0 0 0" />
-			<geometry>
-				<cylinder length="0.05" radius="0.05"/>
-			</geometry>
-			<material name="black"/>
-		</visual> -->
-		<collision>
-			<origin xyz="-0.06 0.0 -0.04" rpy="0 0 0" />
-			<geometry>
-				<cylinder length="0.01" radius="0.05"/>
-			</geometry>
-		</collision>
-        <visual>
-			<origin rpy="${PI/2} 0 0" xyz="0.07 -0.013 -0.04" />
-            <geometry>
-                <mesh filename="file://${mesh_lidar}" />
-            </geometry>
-        </visual>
-		<![CDATA[
-        <collision>
-			<origin rpy="0 0 0" xyz="0 0 0" />
-			<!-- <geometry>
-				<box size="1000 1000 0.01" />
-			</geometry> -->
-			<geometry>
-				<!-- <mesh filename="file://${mesh_lidar}" /> -->
-				<!-- <box size="0.01 0.01 0.01" /> -->
-				<cylinder length="0.01" radius="0.5" />
-			</geometry>
-        </collision>
-        <!-- <inertial_cylinder mass="0.1" length="0.04" radius="0.05">
-            <origin xyz="0 0 0" rpy="0 0 0"/>
-        </inertial_cylinder> -->
-		<inertial>
-			<origin rpy="0 0 0" xyz="0 0 0" />
-			<mass value="0.000" />
-			<inertia ixx="0.166667" ixy="0" ixz="0" iyy="0.166667" iyz="0" izz="0.166667" />
-			<!-- ad camera inertia -->
-		</inertial>]]>
-    </link>
-	<!-- JOINTS  -->
-	<joint name="base_to_right_w" type="continuous">
-		<parent link="chassis" />
-		<child link="right_wheel" />
-		<origin xyz="0.05 -0.09 0.0" />
-		<axis xyz="0 1 0" rpy="0 0 0" />
-		<limit effort="100" velocity="100"/>
-		<joint_properties damping="0.0" friction="0.0"/>
-	</joint>
-	<joint name="base_to_left_w" type="continuous">
-		<parent link="chassis" />
-		<child link="left_wheel" />
-		<origin xyz="0.05 0.09 0" />
-		<axis xyz="0 1 0" rpy="0 0 0" />
-		<limit
-		effort="100" velocity="100"/>
-		<joint_properties damping="0.0" friction="0.0"/>
-	</joint>
-	<!---->
-	<joint name="camera_to_base" type="fixed">
-		<parent link="chassis" />
-		<child link="camera" />
-		<origin xyz="0.1 0 0.048" rpy="0.0 0 0.0" />
-	</joint>
-	<joint name="camera_frame_to_camera" type="fixed">
-		<origin xyz="0 0 0" rpy="${-pi/2} 0 ${-pi/2}" />
-		<parent link="camera" />
-		<child link="camera_frame_optical" />
-	</joint>
-	<joint name="lidar_to_base" type="fixed">
-        <parent link="chassis"/>
-        <child link="lidar"/>
-        <origin xyz="0.05 0 0.115" rpy="0 0 ${PI}"/>
-    </joint>
-	<!-- TRANSMISSIONS (For a more complex model and it represents actuator attributes) -->
-	<transmission name="right_wheel_trans">
-		<type>transmission_interface/SimpleTransmission</type>
-		<joint name="base_to_right_w">
-			<hardwareInterface>hardware_interface/VelocityJointInterface</hardwareInterface>
-		</joint>
-		<actuator name="right_wheel_motor">
-			<mechanicalReduction>34</mechanicalReduction>
-			<hardwareInterface>hardware_interface/EffortJointInterface</hardwareInterface>
-		</actuator>
-	</transmission>
-	<transmission name="left_wheel_trans">
-		<type>transmission_interface/SimpleTransmission</type>
-		<joint name="base_to_left_w">
-			<hardwareInterface>hardware_interface/VelocityJointInterface</hardwareInterface>
-		</joint>
-		<actuator name="left_wheel_motor">
-			<mechanicalReduction>34</mechanicalReduction>
-			<hardwareInterface>hardware_interface/EffortJointInterface</hardwareInterface>
-		</actuator>
-	</transmission>
+    <!-- Place chassis -->
+    <xacro:chassis/>
+    <!-- Add wheels -->
+    <xacro:wheel prefix="left" rot="${rpy_left_wheel}" origin="${origin_left_wheel}"/>
+    <xacro:wheel prefix="right" rot="${rpy_right_wheel}" origin="${origin_right_wheel}"/>
+    <!-- Add camera -->
+    <xacro:camera/>
+    <!-- LIDAR-->
+    <xacro:lidar/>
 </robot>
