Commit message: Added Rviz visualization and improved launch files

File: ros_ws/src/simulation/urdf/wombat.xacro (robot description, xacro)
@@ -14,4 +14,5 @@
 		<parent link="base_link" />
 		<child link="chassis" />
+        <origin xyz="0.0 0.0 ${wheelRadius+0.0010032}" />
 	</joint>
 	<link name="chassis">

Commit message: Linked robot to odometry in rviz and improved ROS structure

File: ros_ws/src/simulation/urdf/wombat.xacro (robot description, xacro)
@@ -10,12 +10,11 @@
     <xacro:include filename="$(find simulation)/urdf/lidar.xacro"/>
     <xacro:include filename="$(find simulation)/urdf/chassis.xacro"/>
-	<!-- Dummy link to fiz robot chassis -->
+    <!-- Dummy link to fiz robot chassis -->
 	<link name="base_link">
-		<pose>0 0 0 0 0 0</pose>
 	</link>
 	<joint name="base_link_to_chassis" type="fixed">
 		<parent link="base_link" />
 		<child link="chassis" />
-        <origin xyz="0.0 0.0 ${wheelRadius+0.0010032}" />
+        <origin xyz="0.0 0.0 0.0"/>
 	</joint>
     <!-- Place chassis -->
